File: HW/reactor.brd (EAGLE design)
At the start: 64.5 x 45.7 mm, 9 parts

Commit message: Finished design
Parts:
- removed C1: (no value), rcl:C0603
- removed LED1: (no value), led:CHIP-LED0603
- removed U$2: (no value), BoneCapeParts:LGA14
- removed U$3: (no value), BoneCapeParts:LGA28-4X5
- removed U$4: (no value), BoneCapeParts:LGA28
- added C10, C14, C15, C17, C19, C2, C3, C6, C9: 0.1u, rcl:C0603
- added C11, C7: 0.22u, rcl:C0603
- added C12, C5: 4.7u, rcl:C0603
- added C13, C18, C4, C8: 10u, rcl:C0603
- added C16: 10n, rcl:C0603
- added R10, R9: 10K, DNI, rcl:R0603
- added R11, R12, R13, R14, R15, R16, R17, R18, R19, R20, R21, R22, R4, R5, R6: 33, rcl:R0603
- added R2: 5.6K, 5%, rcl:R0603
- added R3, R7, R8: 10K, rcl:R0603
- added U$7: (no value), BoneCapeParts:LGA14
- added U$8: (no value), BoneCapeParts:LGA28-4X5
- added U$9: (no value), BoneCapeParts:LGA28
- R1: value (none) -> 5.6K, 5%
- moved R1 96.4 mm to (66.7, 21.0), flipped to the bottom
- moved U$6 74.3 mm to (50.2, 15.9)
- moved U$5 73.9 mm to (50.2, 24.8)
Connections:
- net 5V renamed +5V
- removed net VCC: U$1.VCC
- removed net VDD: U$5.5, U$6.VDD
- new net +3V3: C10.1, C13.1, C14.1, C15.1, C17.1, C19.1, C3.1, C4.1, C6.1, C8.1, C9.1, R1.2, R2.1, R3.2, R4.2, R7.1, R8.1, U$1.VCC, U$5.5, U$6.ANODE_E, U$7.1, U$7.14, U$8.10, U$8.11, U$8.12, U$8.13, U$8.14, U$8.16, U$8.21, U$8.22, U$8.23, U$8.25, U$8.26, U$8.7, U$8.8, U$8.9, U$9.10, U$9.11, U$9.12, U$9.16, U$9.21, U$9.22, U$9.23, U$9.25, U$9.27, U$9.8, U$9.9
- new net DRDY: R20.1, U$7.9
- new net I2C_SCL: R2.2, R21.1, R6.2, U$6.SCL, U$7.2, U$8.24, U$9.24
- new net I2C_SDA: R1.1, R22.1, R5.2, U$6.SDA, U$7.3, U$8.28, U$9.28
- new net INT1: R11.2, U$7.5
- new net INT1_A/M: R19.1, U$8.20, U$9.20
- new net INT1_G: R16.1, U$8.18, U$9.17
- new net INT_IR: R18.2, R3.1, U$6.INT
- new net N$1: C18.1, C2.1, R4.1, U$6.VDD
- new net N$10: R12.2, U$1.TIM@10
- new net N$12: R15.2, U$1.GPIO@4
- new net N$13: R14.2, U$1.GPIO@5
- new net N$14: R13.2, U$1.GPIO@6
- new net N$18: R17.2, U$1.TIM_OUT
- new net N$19: R16.2, U$1.GPIO_INT@2
- new net N$2: R18.1, U$1.GPIO_INT@1
- new net N$3: R11.1, U$1.GPIO@1
- new net N$4: R19.2, U$1.TIM@9
- new net N$45: C7.1, U$7.12
- new net N$46: C7.2, U$7.13
- new net N$47: C5.1, U$7.6
- new net N$48: C16.1, U$8.15
- new net N$5: R20.2, U$1.TIM@8
- new net N$50: C11.1, U$9.13
- new net N$51: C11.2, C12.2, U$9.14
- new net N$52: C12.1, U$9.5
- new net N$6: R6.1, U$1.GPIO@2
- new net N$7: R5.1, U$1.GPIO@3
- new net N$8: R21.2, U$1.SPIB_SOMI/I2C_SCL
- new net N$9: R22.2, U$1.SPIB_SIMO/I2C_SDA
- new net RGB_OUT: R17.1, U$5.6
- new net RGB_S0: R13.1, R7.2, R8.2, U$5.1
- new net RGB_S1: R10.1, R12.1, R9.1, U$5.2
- new net RGB_S2: R15.1, U$5.7
- new net RGB_S3: R14.1, U$5.8
- net GND: now also C10.2, C13.2, C14.2, C15.2, C16.2, C17.2, C18.2, C19.2, C2.2, C3.2, C4.2, C5.2, C6.2, C8.2, C9.2, R10.2, R9.2, U$5.3, U$6.CATHODE_E, U$7.10, U$7.11, U$7.7, U$8.1, U$8.2, U$8.27, U$8.3, U$8.4, U$8.5, U$8.6, U$9.1, U$9.2, U$9.26, U$9.3, U$9.4, U$9.6, U$9.7
Routing:
- net +3V3: track 0.00 -> 146.4 mm, vias 0 -> 12
- net GND: track 0.00 -> 138.0 mm, vias 0 -> 11
- net I2C_SCL: track 0.00 -> 100.7 mm, vias 0 -> 4
- net I2C_SDA: track 0.00 -> 85.5 mm, vias 0 -> 8
- net INT1_G: track 0.00 -> 64.5 mm, vias 0 -> 2
- net INT1_A/M: track 0.00 -> 42.9 mm, vias 0 -> 6
- net RGB_OUT: track 0.00 -> 40.7 mm, vias 0 -> 1
- net INT1: track 0.00 -> 39.8 mm, vias 0 -> 4
- net RGB_S0: track 0.00 -> 32.1 mm, vias 0 -> 5
- net RGB_S1: track 0.00 -> 31.9 mm, vias 0 -> 3
- net RGB_S3: track 0.00 -> 26.9 mm, vias 0 -> 1
- net RGB_S2: track 0.00 -> 25.0 mm, vias 0 -> 3
- net INT_IR: track 0.00 -> 21.4 mm, vias 0 -> 4
- net N$1: track 0.00 -> 10.5 mm, vias 0 -> 2
- net DRDY: track 0.00 -> 10.0 mm, vias 0 -> 3
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Other:
- board size 64.5 x 45.7 mm -> 50.8 x 34.3 mm
- board text added: "Reactor"
- board text removed: "Interacto"
