File: HW/reactor.sch (EAGLE design)
At the start: 9 parts

Commit message: Finished design
Parts:
- removed C1: (no value), rcl:C-EUC0603
- removed LED1: (no value), led:LEDCHIP-LED0603
- removed U$2: (no value), BoneCapeParts:LSM303DLHC
- removed U$3: (no value), BoneCapeParts:LSM330DLC
- removed U$4: (no value), BoneCapeParts:LSM333D
- added C10, C14, C15, C17, C19, C2, C3, C6, C9: 0.1u, rcl:C-EUC0603
- added C11, C7: 0.22u, rcl:C-EUC0603
- added C12, C5: 4.7u, rcl:C-EUC0603
- added C13, C18, C4, C8: 10u, rcl:C-EUC0603
- added C16: 10n, rcl:C-EUC0603
- added R10, R9: 10K, DNI, rcl:R-US_R0603
- added R11, R12, R13, R14, R15, R16, R17, R18, R19, R20, R21, R22, R4, R5, R6: 33, rcl:R-US_R0603
- added R2: 5.6K, 5%, rcl:R-US_R0603
- added R3, R7, R8: 10K, rcl:R-US_R0603
- added U$7: (no value), BoneCapeParts:LSM303DLHC
- added U$8: (no value), BoneCapeParts:LSM330DLC
- added U$9: (no value), BoneCapeParts:LSM333D
- R1: value (none) -> 5.6K, 5%; MPN (none) -> RK73B1JTTDD562J
- U$5: MPN (none) -> TCS32X0
- U$6: MPN (none) -> VCNL3020
Connections:
- new net +3V3: C10.1, C13.1, C14.1, C15.1, C17.1, C19.1, C3.1, C4.1, C6.1, C8.1, C9.1, R1.2, R2.1, R3.2, R4.2, R7.1, R8.1, U$1.VCC, U$5.VDD, U$6.IR_AN, U$7.VDD, U$7.VDD_IO, U$8.CS_A, U$8.CS_G, U$8.DEN_G, U$8.SD0_G/SA0, U$8.VDD@1, U$8.VDD@2, U$8.VDD@3, U$8.VDD@4, U$8.VDD@5, U$8.VDD@6, U$8.VDD@7, U$8.VDD@8, U$8.VDD_IO@1, U$8.VDD_IO@2, U$9.CS_A/M, U$9.CS_G, U$9.DEN_G, U$9.SDO_A/SA0, U$9.VDD@1, U$9.VDD@2, U$9.VDD@3, U$9.VDD@4, U$9.VDD@5, U$9.VDD_IO@1, U$9.VDD_IO@2
- new net +5V: U$1.5V
- new net DRDY: R20.1, U$7.DRDY
- new net GND: C10.2, C13.2, C14.2, C15.2, C16.2, C17.2, C18.2, C19.2, C2.2, C3.2, C4.2, C5.2, C6.2, C8.2, C9.2, R10.2, R9.2, U$1.GND@1, U$1.GND@2, U$5.!OE, U$5.GND, U$6.GND, U$6.IR_CATH, U$7.GND@1, U$7.GND@2, U$7.GND@3, U$8.GND@1, U$8.GND@2, U$8.GND@3, U$8.GND@4, U$8.GND@5, U$8.GND@6, U$8.SD0_A/SA0, U$9.GND@1, U$9.GND@2, U$9.GND@3, U$9.GND@4, U$9.GND@5, U$9.GND@6, U$9.SDO_G/SA0
- new net I2C_SCL: R2.2, R21.1, R6.2, U$6.SCL, U$7.SCL, U$8.SCL_A/G, U$9.SCL/SPC
- new net I2C_SDA: R1.1, R22.1, R5.2, U$6.SDA, U$7.SDA, U$8.SDA_A/G, U$9.SDA
- new net INT1: R11.2, U$7.INT1
- new net INT1_A/M: R19.1, U$8.INT1_A, U$9.INT1_A/M
- new net INT1_G: R16.1, U$8.INT1_G, U$9.INT1_G
- new net INT_IR: R18.2, R3.1, U$6.INT
- new net N$1: C18.1, C2.1, R4.1, U$6.VDD
- new net N$10: R12.2, U$1.TIM@10
- new net N$12: R15.2, U$1.GPIO@4
- new net N$13: R14.2, U$1.GPIO@5
- new net N$14: R13.2, U$1.GPIO@6
- new net N$18: R17.2, U$1.TIM_OUT
- new net N$19: R16.2, U$1.GPIO_INT@2
- new net N$2: R18.1, U$1.GPIO_INT@1
- new net N$3: R11.1, U$1.GPIO@1
- new net N$4: R19.2, U$1.TIM@9
- new net N$45: C7.1, U$7.SETP
- new net N$46: C7.2, U$7.SETC
- new net N$47: C5.1, U$7.C1
- new net N$48: C16.1, U$8.CAP
- new net N$5: R20.2, U$1.TIM@8
- new net N$50: C11.1, U$9.SETC
- new net N$51: C11.2, C12.2, U$9.SETP
- new net N$52: C12.1, U$9.C1
- new net N$6: R6.1, U$1.GPIO@2
- new net N$7: R5.1, U$1.GPIO@3
- new net N$8: R21.2, U$1.SPIB_SOMI/I2C_SCL
- new net N$9: R22.2, U$1.SPIB_SIMO/I2C_SDA
- new net RGB_OUT: R17.1, U$5.OUT
- new net RGB_S0: R13.1, R7.2, R8.2, U$5.S0
- new net RGB_S1: R10.1, R12.1, R9.1, U$5.S1
- new net RGB_S2: R15.1, U$5.S2
- new net RGB_S3: R14.1, U$5.S3
Other:
- note added: "0x13"
- note added: "0x18"
- note added: "0x19"
- note added: "0x1D"
- note added: "0x1E"
- note added: "0x6A"
- note added: "0x6B"
- moved on the sheet: R1, U$1, U$5, U$6
